Commit message: Add gazebo launch file and update URDF with inertial properties and collision elements

File: src/agv_description/urdf/agv_gazebo.xacro (robot description, xacro)
@@ -2,10 +2,28 @@
 <robot name="agv" xmlns="http://www.ros.org/wiki/xacro">
     <gazebo reference = "wheel_right_link">
-        <material>Gazebo/Black</material>
-        <mu1>100.0</mu1>
-        <mu2>100.0</mu2>
-        <friction>100.0</friction>
-        <rolling_friction>0.01</rolling_friction>
-        <restitution_coefficient>0.1</restitution_coefficient>
+        <mu1>100000000000000.0</mu1>
+        <mu2>100000000000000.0</mu2>
+        <kp>1000000000000.0</kp>
+        <kd>10000000000.0</kd>
+        <minDepth>0.001</minDepth>
+        <maxVel>0.1</maxVel>
+        <fdir1>1 0 0</fdir1>
+    </gazebo>
+    <gazebo reference = "wheel_left_link">
+        <mu1>100000000000000.0</mu1>
+        <mu2>100000000000000.0</mu2>
+        <kp>1000000000000.0</kp>
+        <kd>10000000000.0</kd>
+        <minDepth>0.001</minDepth>
+        <maxVel>0.1</maxVel>
+        <fdir1>1 0 0</fdir1>
+    </gazebo>
+    <gazebo reference = "caster_link">
+        <mu1>0.1</mu1>
+        <mu2>0.1</mu2>
+        <kp>1000000.0</kp>
+        <kd>100.0</kd>
+        <minDepth>0.001</minDepth>
+        <maxVel>0.1</maxVel>
     </gazebo>
 </robot>
