Commit message: feat: overhaul robot description with updated CAD meshes and structured URDF configuration. Support gazebo sim

File: src/agv_description/urdf/agv_gazebo.xacro (robot description, xacro)
@@ -1,53 +1,159 @@
 <?xml version="1.0"?>
-<robot name="agv" xmlns:xacro="http://ros.org/wiki/xacro">
-    <gazebo reference = "wheel_right_link">
+<robot xmlns:xacro="http://www.ros.org/wiki/xacro">
+    <!-- ==================== GAZEBO PROPERTIES ==================== -->
+    <gazebo reference="base_link-v3">
+        <material>Gazebo/DarkGrey</material>
+    </gazebo>
+    <gazebo reference="wheel_bracket_left-v4">
+        <material>Gazebo/Grey</material>
+    </gazebo>
+    <gazebo reference="wheel_bracket_right-v1">
+        <material>Gazebo/Grey</material>
+    </gazebo>
+    <gazebo reference="wheel_left-v2">
+        <material>Gazebo/FlatBlack</material>
         <mu1>1.0</mu1>
         <mu2>1.0</mu2>
-        <!-- <mu1>100000000000000.0</mu1>
-        <mu2>100000000000000.0</mu2> -->
-        <!-- <mu1>0.5</mu1>
-        <mu2>0.5</mu2> -->
-        <!-- <kp>1000000000000.0</kp> -->
-        <kp>100000.0</kp>
-        <!-- <kd>10000000000.0</kd> -->
-        <kd>100.0</kd>
+        <kp>1000000.0</kp>
+        <kd>1.0</kd>
         <minDepth>0.001</minDepth>
-        <maxVel>1.0</maxVel>
-        <fdir1>1 0 0</fdir1>
     </gazebo>
-    <gazebo reference = "wheel_left_link">
+    <gazebo reference="wheel_right-v1">
+        <material>Gazebo/FlatBlack</material>
         <mu1>1.0</mu1>
         <mu2>1.0</mu2>
-        <!-- <mu1>100000000000000.0</mu1>
-        <mu2>100000000000000.0</mu2> -->
-        <!-- <kp>1000000000000.0</kp>
-        <kd>10000000000.0</kd> -->
-        <!-- <mu1>0.5</mu1>
-        <mu2>0.5</mu2> -->
-        <kp>100000.0</kp>
-        <kd>100.0</kd>
+        <kp>1000000.0</kp>
+        <kd>1.0</kd>
         <minDepth>0.001</minDepth>
-        <maxVel>1.0</maxVel>
-        <fdir1>1 0 0</fdir1>
     </gazebo>
-    <gazebo reference = "caster_link">
-        <mu1>0.001</mu1>
-        <mu2>0.001</mu2>
+    <gazebo reference="castrol_bracket_left-v2">
+        <material>Gazebo/Grey</material>
+    </gazebo>
+    <gazebo reference="castrol_bracket_right-v1">
+        <material>Gazebo/Grey</material>
+    </gazebo>
+    <gazebo reference="castrol_housing_left_link-v3">
+        <material>Gazebo/Grey</material>
+    </gazebo>
+    <gazebo reference="castrol_housing_right_link-v1">
+        <material>Gazebo/Grey</material>
+    </gazebo>
+    <gazebo reference="castrol_yaw_link_left-v3">
+        <material>Gazebo/Grey</material>
+    </gazebo>
+    <gazebo reference="castrol_yaw_link_right-v1">
+        <material>Gazebo/Grey</material>
+    </gazebo>
+    <gazebo reference="castrol_wheel_left-v2">
+        <material>Gazebo/FlatBlack</material>
+        <mu1>0.05</mu1>
+        <mu2>0.05</mu2>
         <kp>1000000.0</kp>
-        <kd>100.0</kd>
-        <minDepth>0.001</minDepth>
-        <maxVel>0.1</maxVel>
+        <kd>1.0</kd>
     </gazebo>
+    <gazebo reference="castrol_wheel_right-v1">
+        <material>Gazebo/FlatBlack</material>
+        <mu1>0.05</mu1>
+        <mu2>0.05</mu2>
+        <kp>1000000.0</kp>
+        <kd>1.0</kd>
+    </gazebo>
+    <gazebo reference="camera_base-v3">
+        <material>Gazebo/Grey</material>
+    </gazebo>
+    <gazebo reference="lidar_housing-v2">
+        <material>Gazebo/DarkGrey</material>
+    </gazebo>
+    <!-- Lidar Ray Sensor Plugin -->
+    <gazebo reference="lidar_head-v2">
+        <material>Gazebo/Black</material>
+        <sensor type="ray" name="lidar_sensor">
+            <pose>0 0 0 0 0 0</pose>
+            <visualize>false</visualize>
+            <update_rate>10</update_rate>
+            <ray>
+                <scan>
+                    <horizontal>
+                        <samples>360</samples>
+                        <resolution>1</resolution>
+                        <min_angle>-3.14159265</min_angle>
+                        <max_angle>3.14159265</max_angle>
+                    </horizontal>
+                </scan>
+                <range>
+                    <min>0.12</min>
+                    <max>12.0</max>
+                    <resolution>0.01</resolution>
+                </range>
+                <noise>
+                    <type>gaussian</type>
+                    <mean>0.0</mean>
+                    <stddev>0.01</stddev>
+                </noise>
+            </ray>
+            <plugin name="gazebo_ros_lidar" filename="libgazebo_ros_ray_sensor.so">
+                <ros>
+                    <remapping>~/out:=scan</remapping>
+                </ros>
+                <output_type>sensor_msgs/LaserScan</output_type>
+                <frame_name>lidar_head-v2</frame_name>
+            </plugin>
+        </sensor>
+    </gazebo>
+    <!-- IMU Sensor Plugin -->
+    <gazebo reference="imu_link-v1">
+        <material>Gazebo/Red</material>
+        <sensor name="imu_sensor" type="imu">
+            <always_on>true</always_on>
+            <update_rate>100</update_rate>
+            <visualize>false</visualize>
+            <plugin name="gazebo_ros_imu" filename="libgazebo_ros_imu_sensor.so">
+                <ros>
+                    <namespace>/</namespace>
+                    <remapping>~/out:=imu/out</remapping>
+                </ros>
+                <initial_orientation_as_reference>false</initial_orientation_as_reference>
+                <frame_name>imu_link-v1</frame_name>
+            </plugin>
+        </sensor>
+    </gazebo>
+    <!-- ==================== GAZEBO PLUGINS ==================== -->
     <gazebo>
-        <xacro:if value="$(arg is_ignition)">
-            <plugin filename="ign_ros2_control-system" name="ign_ros2_control::IgnitionROS2ControlPlugin">
-                <parameters>$(find agv_controller)/config/agv_controllers.yaml</parameters>
-            </plugin>
-        </xacro:if>
-        <xacro:unless value="$(arg is_ignition)">
-            <plugin filename="gz_ros2_control-system" name="gz_ros2_control::GazeboSimROS2ControlPlugin">
-                <parameters>$(find agv_controller)/config/agv_controllers.yaml</parameters>
-            </plugin>
-        </xacro:unless>
+        <!-- Differential Drive Controller Plugin -->
+        <plugin name="differential_drive_controller" filename="libgazebo_ros_diff_drive.so">
+            <ros>
+                <namespace>/</namespace>
+                <remapping>cmd_vel:=cmd_vel</remapping>
+                <remapping>odom:=odom</remapping>
+            </ros>
+            <update_rate>50</update_rate>
+            <left_joint>wheel_bracket_left-v4_Revolute-3</left_joint>
+            <right_joint>wheel_bracket_right-v1_Revolute-4</right_joint>
+            <wheel_separation>0.30</wheel_separation>
+            <wheel_diameter>0.10</wheel_diameter>
+            <max_wheel_torque>20.0</max_wheel_torque>
+            <max_wheel_acceleration>2.0</max_wheel_acceleration>
+            <command_topic>cmd_vel</command_topic>
+            <publish_odom>true</publish_odom>
+            <publish_odom_tf>true</publish_odom_tf>
+            <publish_wheel_tf>true</publish_wheel_tf>
+            <odometry_topic>odom</odometry_topic>
+            <odometry_frame>odom</odometry_frame>
+            <robot_base_frame>base_footprint</robot_base_frame>
+        </plugin>
+        <!-- Joint State Publisher Plugin -->
+        <plugin name="agv_joint_state" filename="libgazebo_ros_joint_state_publisher.so">
+            <ros>
+                <namespace>/</namespace>
+                <remapping>joint_states:=joint_states</remapping>
+            </ros>
+            <update_rate>50</update_rate>
+            <joint_name>wheel_bracket_left-v4_Revolute-3</joint_name>
+            <joint_name>wheel_bracket_right-v1_Revolute-4</joint_name>
+            <joint_name>castrol_housing_left_link-v3_Revolute-9</joint_name>
+            <joint_name>castrol_housing_right_link-v1_Revolute-10</joint_name>
+            <joint_name>castrol_yaw_link_left-v3_Revolute-11</joint_name>
+            <joint_name>castrol_yaw_link_right-v1_Revolute-12</joint_name>
+        </plugin>
     </gazebo>
 </robot>
