Commit message: Enhance URDF configuration by adding inertial properties and collision elements for links; create gazebo simulation file for wheel interactions.

File: src/agv_description/urdf/agv.urdf.xacro (robot description, xacro)
@@ -1,6 +1,12 @@
 <?xml version="1.0"?>
-<robot xmlns="http://www.ros.org/wiki/xacro" name="agv">
+<robot xmlns:xacro="http://www.ros.org/wiki/xacro" name="agv">
+    <xacro:include filename="$(find agv_description)/urdf/agv_gazebo.xacro"/>
     <link name="base_footprint"/>
     <link name="base_link">
+        <inertial>
+            <origin xyz="0.0 0.0 0.904348"/>
+            <mass value="3.0"/>
+            <inertia ixx="0.02" ixy="0" ixz="0" iyy="0.0325" iyz="0" izz="0.0325" />
+        </inertial>
         <visual>
             <origin rpy="0.0 0.0 0.0" xyz="0.0 0.0 0.0"/>
@@ -9,4 +15,10 @@
             </geometry>
         </visual>
+        <collision>
+            <origin rpy="0.0 0.0 0.0" xyz="0.0 0.0 0.0"/>
+            <geometry>
+                <mesh filename="package://agv_description/meshes/base_link.stl" scale="0.001 0.001 0.001"/>
+            </geometry>
+        </collision>
     </link>
     <joint name="base_joint" type="fixed">
@@ -16,4 +28,9 @@
     </joint>
     <link name="wheel_right_link">
+        <inertial>
+            <origin xyz="0.0 -0.014 0.0" rpy="0.0 0.0 0.0"/>
+            <mass value="0.0530086090966721"/>
+            <inertia ixx="0.00000304" ixy="0.0" ixz="0.0" iyy="0.0000052" iyz="0.0" izz="0.00000304"/>
+        </inertial>
         <visual>
             <origin rpy="1.570796 0.0 0.0" xyz="0.0 0.0 0.0"/>
@@ -22,4 +39,10 @@
             </geometry>
         </visual>
+        <collision>
+            <origin rpy="1.570796 0.0 0.0" xyz="0.0 0.0 0.0"/>
+            <geometry>
+                <mesh filename="package://agv_description/meshes/wheel_right_link.stl" scale="0.001 0.001 0.001"/>
+            </geometry>
+        </collision>
     </link>
     <joint name="wheel_right_joint" type="continuous">
@@ -30,6 +53,10 @@
     </joint>
     <link name="wheel_left_link">
+        <inertial>
+            <origin xyz="0.0 0.014 0.0" rpy="0.0 0.0 0.0"/>
+            <mass value="0.0530086090966721"/>
+            <inertia ixx="0.00000304" ixy="0.0" ixz="0.0" iyy="0.0000052" iyz="0.0" izz="0.00000304"/>
+        </inertial>
         <visual>
-            <!-- -1.57 0.0 1.57  1.8 1.3 0.0-->
             <origin rpy="1.570796 0.0 0.0" xyz="0.0 0.0 0.0"/>
             <geometry>
@@ -37,4 +64,10 @@
             </geometry>
         </visual>
+        <collision>
+            <origin rpy="1.570796 0.0 0.0" xyz="0.0 0.0 0.0"/>
+            <geometry>
+                <mesh filename="package://agv_description/meshes/wheel_right_link.stl" scale="0.001 0.001 0.001"/>
+            </geometry>
+        </collision>
     </link>
     <joint name="wheel_left_joint" type="continuous">
@@ -45,4 +78,9 @@
     </joint>
     <link name="caster_link">
+        <inertial>
+            <origin xyz="0.0 0.0 0.0" rpy="0.0 0.0 0.0"/>
+            <mass value="0.1"/>
+            <inertia ixx="0.0001" ixy="0.0" ixz="0.0" iyy="0.0001" iyz="0.0" izz="0.0001"/>
+        </inertial>
         <visual>
             <origin rpy="0.0 0.0 0.0" xyz="0.0 0.0 0.0"/>
@@ -51,4 +89,10 @@
             </geometry>
         </visual>
+        <collision>
+            <origin xyz="0.0 0.0 0.0"/>
+            <geometry>
+                <mesh filename="package://agv_description/meshes/caster_link.stl" scale="0.001 0.001 0.001"/>
+            </geometry>
+        </collision>
     </link>
     <joint name="caster_joint" type="fixed">

Commit message: URDF pakai versi bumperbot sementara, joystick sudah bisa tapi belum differetial drive

File: src/agv_description/urdf/agv.urdf.xacro (robot description, xacro)
@@ -4,115 +4,173 @@
     <!-- Include Gazebo Parameters-->
     <xacro:include filename="$(find agv_description)/urdf/agv_gazebo.xacro"/>
+     <!-- Load Simulated or Real Hardware Interfaces -->
+    <xacro:arg name="is_sim" default="true"/>
     <!-- ROS 2 Control -->
     <xacro:include filename="$(find agv_description)/urdf/agv_ros2_control.xacro"/>
     <link name="base_footprint"/>
-    <link name="base_link">
-        <inertial>
-            <origin xyz="0.0 0.0 0.904348"/>
-            <!-- <mass value="3.0"/>
-            <inertia ixx="0.02" ixy="0" ixz="0" iyy="0.0325" iyz="0" izz="0.0325" /> -->
-            <mass value="8.2573504e-01"/>
-            <inertia ixx="2.2124416e-02" ixy="-1.2294101e-04" ixz="3.4938785e-04" iyy="2.1193702e-02" iyz="-5.0120904e-05" izz="2.0064271e-02"/>
-        </inertial>
-        <visual>
-            <origin rpy="0.0 0.0 0.0" xyz="0.0 0.0 0.0"/>
-            <geometry>
-                <mesh filename="package://agv_description/meshes/base_link.stl" scale="0.001 0.001 0.001"/>
-            </geometry>
-        </visual>
-        <collision>
-            <origin rpy="0.0 0.0 0.0" xyz="0.0 0.0 0.0"/>
-            <geometry>
-                <mesh filename="package://agv_description/meshes/base_link.stl" scale="0.001 0.001 0.001"/>
-            </geometry>
-        </collision>
-    </link>
-    <joint name="base_joint" type="fixed">
-        <parent link="base_footprint"/>
-        <child link="base_link"/>
-        <origin rpy="0.0 0.0 0.0" xyz="0.0 0.0 0.315"/>
-    </joint>
-    <link name="wheel_right_link">
-        <inertial>
-            <origin xyz="0.0 -0.014 0.0" rpy="0.0 0.0 0.0"/>
-            <!-- <mass value="0.0530086090966721"/>
-            <inertia ixx="0.00000304" ixy="0.0" ixz="0.0" iyy="0.0000052" iyz="0.0" izz="0.00000304"/> -->
-            <mass value="0.0530086090966721"/>
-            <inertia ixx="1.88176298336665E-05" ixy="-4.8444933029987E-10" ixz="1.88163708851143E-08" iyy="3.11510738647764E-05" iyz="-6.93560663069607E-11" izz="1.8801969558182E-05"/>
-        </inertial>
-        <visual>
-            <origin rpy="1.570796 0.0 0.0" xyz="0.0 0.0 0.0"/>
-            <geometry>
-                <mesh filename="package://agv_description/meshes/wheel_right_link.stl" scale="0.001 0.001 0.001"/>
-            </geometry>
-        </visual>
-        <collision>
-            <origin rpy="1.570796 0.0 0.0" xyz="0.0 0.0 0.0"/>
-            <geometry>
-                <mesh filename="package://agv_description/meshes/wheel_right_link.stl" scale="0.001 0.001 0.001"/>
-                <!-- <sphere radius="0.300"/> -->
-            </geometry>
-        </collision>
-    </link>
-    <joint name="wheel_right_joint" type="continuous">
-        <parent link="base_link"/>
-        <child link="wheel_right_link"/>
-        <axis xyz="0.0 1.0 0.0"/>
-        <origin rpy="0.0 0.0 -1.570796" xyz="-1.55 1.22 0.0"/>
-    </joint>
-    <link name="wheel_left_link">
-        <inertial>
-            <origin xyz="0.0 0.014 0.0" rpy="0.0 0.0 0.0"/>
-            <!-- <mass value="0.0530086090966721"/>
-            <inertia ixx="0.00000304" ixy="0.0" ixz="0.0" iyy="0.0000052" iyz="0.0" izz="0.00000304"/> -->
-            <mass value="0.0530086043217644"/>
-            <inertia ixx="1.8792911368909E-05" ixy="3.31256392204584E-10" ixz="-1.14082001662767E-08" iyy="3.11510738759073E-05" iyz="-3.60499245082192E-10" izz="1.88266886146847E-05"/>
-        </inertial>
-        <visual>
-            <origin rpy="-1.570796 0.0 0.0" xyz="0.0 0.0 0.0"/>
-            <geometry>
-                <mesh filename="package://agv_description/meshes/wheel_right_link.stl" scale="0.001 0.001 0.001"/>
-            </geometry>
-        </visual>
-        <collision>
-            <origin rpy="1.570796 0.0 0.0" xyz="0.0 0.0 0.0"/>
-            <geometry>
-                <mesh filename="package://agv_description/meshes/wheel_right_link.stl" scale="0.001 0.001 0.001"/>
-                 <!-- <sphere radius="0.300"/> -->
-            </geometry>
-        </collision>
-    </link>
-    <joint name="wheel_left_joint" type="continuous">
-        <parent link="base_link"/>
-        <child link="wheel_left_link"/>
-        <axis xyz="0.0 1.0 0.0"/>
-        <origin rpy="0.0 0.0 -1.570796" xyz="1.55 1.22 0.0"/>
-    </joint>
-    <link name="caster_link">
-        <inertial>
-            <origin xyz="0.0 0.0 0.0" rpy="0.0 0.0 0.0"/>
-            <!-- <mass value="0.1"/>
-            <inertia ixx="0.0001" ixy="0.0001" ixz="0.0001" iyy="0.0001" iyz="0.0001" izz="0.0001"/> -->
-            <mass value="1.44379265037903E-06"/>
-            <inertia ixx="7.23075276010246E-11" ixy="-6.10956883467859E-16" ixz="2.22849693525031E-15" iyy="3.8713793085917E-11" iyz="2.93909858781952E-15" izz="1.00967486676306E-10"/>
-        </inertial>
-        <visual>
-            <origin rpy="0.0 0.0 0.0" xyz="0.0 0.0 0.0"/>
-            <geometry>
-                <mesh filename="package://agv_description/meshes/caster_link.stl" scale="0.001 0.001 0.001"/>
-            </geometry>
-        </visual>
-        <collision>
-            <origin xyz="0.0 0.0 0.0"/>
-            <geometry>
-                <mesh filename="package://agv_description/meshes/caster_link.stl" scale="0.001 0.001 0.001"/>
-            </geometry>
-        </collision>
-    </link>
-    <joint name="caster_joint" type="fixed">
-        <parent link="base_link"/>
-        <child link="caster_link"/>
-        <axis xyz="0.0 0.0 0.0"/>
-        <origin rpy="0.0 0.0 0.0" xyz="0.0 -0.95 -0.261"/>
-    </joint>
+  <link name="base_link">
+    <inertial>
+      <origin xyz="0 0 0.04" rpy="0.0 0.25 0.3" />
+      <mass value="8.2573504e-01"/>
+      <inertia ixx="2.2124416e-02" ixy="-1.2294101e-04" ixz="3.4938785e-04"
+               iyy="2.1193702e-02" iyz="-5.0120904e-05"
+               izz="2.0064271e-02" />
+    </inertial>
+    <visual>
+      <origin xyz="0 0 0" rpy="0 0 0" />
+      <geometry>
+        <mesh filename="package://agv_description/meshes/base_link.STL" />
+      </geometry>
+    </visual>
+    <collision>
+      <origin xyz="0 0 0" rpy="0 0 0" />
+      <geometry>
+        <mesh filename="package://agv_description/meshes/base_link.STL" />
+      </geometry>
+    </collision>
+  </link>
+  <joint name="base_joint" type="fixed">
+    <parent link="base_footprint"/>
+    <child link="base_link" />
+    <origin xyz="0 0 0.033" rpy="0 0 0"/>
+  </joint>
+  <link name="wheel_right_link">
+    <inertial>
+      <origin xyz="0 -0.014 0" rpy="0 0 0" />
+      <mass value="0.0530086090966721" />
+      <inertia ixx="1.88176298336665E-05" ixy="-4.8444933029987E-10" ixz="1.88163708851143E-08"
+               iyy="3.11510738647764E-05" iyz="-6.93560663069607E-11"
+               izz="1.8801969558182E-05" />
+    </inertial>
+    <visual>
+      <origin xyz="0 0 0" rpy="1.57 0 0" />
+      <geometry>
+        <mesh filename="package://agv_description/meshes/wheel_right_link.STL" />
+      </geometry>
+    </visual>
+    <collision>
+      <origin xyz="0 -0.015 0" rpy="1.57 0 0" />
+      <geometry>
+        <sphere radius="0.033"/>
+      </geometry>
+    </collision>
+  </link>
+  <joint name="wheel_right_joint" type="continuous">
+    <origin xyz="0 -0.0701101849418637 0" rpy="0 0 0" />
+    <parent link="base_link" />
+    <child link="wheel_right_link" />
+    <axis xyz="0 1 0" />
+  </joint>
+  <link
+    name="wheel_left_link">
+    <inertial>
+      <origin xyz="0 0.014 0" rpy="0 0 0" />
+      <mass value="0.0530086043217644" />
+      <inertia ixx="1.8792911368909E-05"  ixy="3.31256392204584E-10" ixz="-1.14082001662767E-08"
+               iyy="3.11510738759073E-05" iyz="-3.60499245082192E-10"
+               izz="1.88266886146847E-05" />
+    </inertial>
+    <visual>
+      <origin xyz="0 0 0" rpy="-1.57 0 0" />
+      <geometry>
+        <mesh filename="package://agv_description/meshes/wheel_left_link.STL" />
+      </geometry>
+    </visual>
+    <collision>
+      <origin xyz="0 0.015 0" rpy="-1.57 0 0" />
+      <geometry>
+        <sphere radius="0.033"/>
+      </geometry>
+    </collision>
+  </link>
+  <joint name="wheel_left_joint" type="continuous">
+    <origin xyz="0 0.0701101849418642 0" rpy="0 0 0" />
+    <parent link="base_link" />
+    <child link="wheel_left_link" />
+    <axis xyz="0 1 0" />
+  </joint>
+  <link name="caster_front_link">
+    <inertial>
+      <origin xyz="3.89968128948481E-07 2.40073004698083E-07 0.00219173397061506" rpy="0 0 0" />
+      <mass value="1.44379265037903E-06" />
+      <inertia ixx="7.23075276010246E-11" ixy="-6.10956883467859E-16" ixz="2.22849693525031E-15"
+               iyy="3.8713793085917E-11"  iyz="2.93909858781952E-15"
+               izz="1.00967486676306E-10" />
+    </inertial>
+    <visual>
+      <origin xyz="0 0 0" rpy="0 0 0" />
+      <geometry>
+        <mesh filename="package://agv_description/meshes/caster_front_link.STL" />
+      </geometry>
+    </visual>
+    <collision>
+      <origin xyz="0 0 0" rpy="0 0 0" />
+      <geometry>
+        <sphere radius="0.005"/>
+      </geometry>
+    </collision>
+  </link>
+  <joint name="caster_front_joint" type="fixed">
+    <origin xyz="0.04755 0 -0.0275" rpy="0 0 0" />
+    <parent link="base_link" />
+    <child link="caster_front_link" />
+    <axis xyz="0 0 0" />
+  </joint>
+  <link name="caster_rear_link">
+    <inertial>
+      <origin xyz="3.8996812895542E-07 2.40073004698083E-07 0.00219173397061509" rpy="0 0 0" />
+      <mass value="1.44379265037902E-06" />
+      <inertia ixx="7.23075276010246E-11" ixy="-6.10956872363424E-16" ixz="2.22849693527207E-15"
+               iyy="3.87137930859167E-11" iyz="2.939098587861E-15"
+               izz="1.00967486676306E-10" />
+    </inertial>
+    <visual>
+      <origin xyz="0 0 0" rpy="0 0 0" />
+      <geometry>
+        <mesh filename="package://agv_description/meshes/caster_rear_link.STL" />
+      </geometry>
+    </visual>
+    <collision>
+      <origin xyz="0 0 0" rpy="0 0 0" />
+      <geometry>
+        <sphere radius="0.005"/>
+      </geometry>
+    </collision>
+  </link>
+  <joint name="caster_rear_joint" type="fixed">
+    <origin xyz="-0.04755 0 -0.0275" rpy="0 0 0" />
+    <parent link="base_link" />
+    <child link="caster_rear_link" />
+    <axis xyz="0 0 0" />
+  </joint>
+  <link name="imu_link">
+    <inertial>
+      <origin xyz="-0.00552433659106688 0.000168210391520346 0.000514000497342681" rpy="0 0 0" />
+      <mass value="0.000528415362211671" />
+      <inertia ixx="1.46176048428261E-08" ixy="1.40015117949421E-10" ixz="-1.99633872937403E-12"
+               iyy="8.59662482954888E-09" iyz="7.52375112767959E-12"
+               izz="2.30279421279312E-08" />
+    </inertial>
+    <visual>
+      <origin xyz="0 0 0" rpy="0 0 0" />
+      <geometry>
+        <mesh filename="package://agv_description/meshes/imu_link.STL" />
+      </geometry>
+      <material name="">
+        <color rgba="0.792156862745098 0.819607843137255 0.933333333333333 1" />
+      </material>
+    </visual>
+    <collision>
+      <origin xyz="0 0 0" rpy="0 0 0" />
+      <geometry>
+        <mesh filename="package://agv_description/meshes/imu_link.STL" />
+      </geometry>
+    </collision>
+  </link>
+  <joint name="imu_joint" type="fixed">
+    <origin xyz="0 0 0.0698986241758014" rpy="0 0 0" />
+    <parent link="base_link" />
+    <child link="imu_link" />
+    <axis xyz="0 0 0" />
+  </joint>
 </robot>

File: src/agv_description/urdf/agv_gazebo.xacro (robot description, xacro)
@@ -2,6 +2,8 @@
 <robot name="agv" xmlns:xacro="http://ros.org/wiki/xacro">
     <gazebo reference = "wheel_right_link">
-        <mu1>100000000000000.0</mu1>
-        <mu2>100000000000000.0</mu2>
+        <mu1>1.0</mu1>
+        <mu2>1.0</mu2>
+        <!-- <mu1>100000000000000.0</mu1>
+        <mu2>100000000000000.0</mu2> -->
         <!-- <mu1>0.5</mu1>
         <mu2>0.5</mu2> -->
@@ -11,10 +13,12 @@
         <kd>100.0</kd>
         <minDepth>0.001</minDepth>
-        <maxVel>0.1</maxVel>
+        <maxVel>1.0</maxVel>
         <fdir1>1 0 0</fdir1>
     </gazebo>
     <gazebo reference = "wheel_left_link">
-        <mu1>100000000000000.0</mu1>
-        <mu2>100000000000000.0</mu2>
+        <mu1>1.0</mu1>
+        <mu2>1.0</mu2>
+        <!-- <mu1>100000000000000.0</mu1>
+        <mu2>100000000000000.0</mu2> -->
         <!-- <kp>1000000000000.0</kp>
         <kd>10000000000.0</kd> -->
@@ -24,5 +28,5 @@
         <kd>100.0</kd>
         <minDepth>0.001</minDepth>
-        <maxVel>0.1</maxVel>
+        <maxVel>1.0</maxVel>
         <fdir1>1 0 0</fdir1>
     </gazebo>
