Commit message: fix: invert yaw rotation of lidar_head_joint in URDF

File: src/agv_description/urdf/agv.xacro (robot description, xacro)
@@ -502,5 +502,5 @@
     </joint>
     <joint name="lidar_head_joint" type="fixed">
-        <origin xyz="0.0 0.0 0.07850000000000001" rpy="0.0 0.0 -1.5707963267948966" />
+        <origin xyz="0.0 0.0 0.07850000000000001" rpy="0.0 0.0 1.5707963267948966" />
         <parent link="lidar_housing-v2" />
         <child link="lidar_head-v2" />

Commit message: chore: update robot base frame to base_footprint and add base_link alias in URDF

File: src/agv_description/urdf/agv.xacro (robot description, xacro)
@@ -511,5 +511,10 @@
         <child link="imu_link-v1" />
     </joint>
-    <!-- ==================== ALIAS FRAMES ==================== -->
+    <link name="base_link" />
+    <joint name="base_link_alias_joint" type="fixed">
+        <parent link="base_link-v3" />
+        <child link="base_link" />
+        <origin xyz="0.0 0.0 0.0" rpy="0.0 0.0 0.0" />
+    </joint>
     <link name="camera_lens_1" />
     <joint name="camera_lens_1_alias_joint" type="fixed">
