Commit message: Revisi urdf visual putar 90 derajat ke kanan. Mapping dengan SLAM Toolbox done

File: src/agv_origin_description/urdf/agv_origin.xacro (robot description, xacro)
@@ -8,5 +8,5 @@
   <parent link="base_footprint"/>
   <child link="base_link"/>
-  <origin xyz="0 0 0.1005" rpy="0 0 0"/>
+  <origin xyz="0 0 0.1005" rpy="0 0 3.14159"/>
 </joint>
 <link name="base_link">
@@ -17,5 +17,5 @@
   </inertial>
   <visual>
-    <origin xyz="0 0 0" rpy="0 0 0"/>
+    <origin xyz="0 0 0" rpy="0 0 -1.5708"/>
     <geometry>
       <mesh filename="file://$(find agv_origin_description)/meshes/base_link.stl" scale="0.001 0.001 0.001"/>
@@ -37,5 +37,5 @@
   </inertial>
   <visual>
-    <origin xyz="-0.0 -0.0 -0.22" rpy="0 0 0"/>
+    <origin xyz="-0.0 -0.0 -0.22" rpy="0 0 -1.5708"/>
     <geometry>
       <mesh filename="file://$(find agv_origin_description)/meshes/lidar_1.stl" scale="0.001 0.001 0.001"/>
@@ -65,5 +65,5 @@
   </inertial>
   <visual>
-    <origin xyz="-0.0 0.115 -0.14" rpy="0 0 0"/>
+    <origin xyz="-0.0 0.115 -0.14" rpy="0 0 -1.5708"/>
     <geometry>
       <mesh filename="file://$(find agv_origin_description)/meshes/depth_cam_1.stl" scale="0.001 0.001 0.001"/>
@@ -85,5 +85,5 @@
   </inertial>
   <visual>
-    <origin xyz="-0.1578 -0.104 0.0435" rpy="0 0 0"/>
+    <origin xyz="-0.1578 -0.104 0.0435" rpy="0 0 -1.5708"/>
     <geometry>
       <mesh filename="file://$(find agv_origin_description)/meshes/left_wheel_1.stl" scale="0.001 0.001 0.001"/>
@@ -105,5 +105,5 @@
   </inertial>
   <visual>
-    <origin xyz="0.1578 -0.104 0.0435" rpy="0 0 0"/>
+    <origin xyz="0.1578 -0.104 0.0435" rpy="0 0 -1.5708"/>
     <geometry>
       <mesh filename="file://$(find agv_origin_description)/meshes/right_wheel_1.stl" scale="0.001 0.001 0.001"/>
@@ -125,5 +125,5 @@
   </inertial>
   <visual>
-    <origin xyz="0.12695 0.1222 0.0406" rpy="0 0 0"/>
+    <origin xyz="0.12695 0.1222 0.0406" rpy="0 0 -1.5708"/>
     <geometry>
       <mesh filename="file://$(find agv_origin_description)/meshes/castrol_bracket_right_1.stl" scale="0.001 0.001 0.001"/>
@@ -145,5 +145,5 @@
   </inertial>
   <visual>
-    <origin xyz="0.109238 0.088 0.075" rpy="0 0 0"/>
+    <origin xyz="0.109238 0.088 0.075" rpy="0 0 -1.5708"/>
     <geometry>
       <mesh filename="file://$(find agv_origin_description)/meshes/castrol_wheel_right_1.stl" scale="0.001 0.001 0.001"/>
@@ -165,5 +165,5 @@
   </inertial>
   <visual>
-    <origin xyz="-0.12695 0.1222 0.0406" rpy="0 0 0"/>
+    <origin xyz="-0.12695 0.1222 0.0406" rpy="0 0 -1.5708"/>
     <geometry>
       <mesh filename="file://$(find agv_origin_description)/meshes/castrol_bracket_left_1.stl" scale="0.001 0.001 0.001"/>
@@ -185,5 +185,5 @@
   </inertial>
   <visual>
-    <origin xyz="-0.109238 0.088 0.075" rpy="0 0 0"/>
+    <origin xyz="-0.109238 0.088 0.075" rpy="0 0 -1.5708"/>
     <geometry>
       <mesh filename="file://$(find agv_origin_description)/meshes/castrol_wheel_left_1.stl" scale="0.001 0.001 0.001"/>

Commit message: update localization berdasarkan map hasil SLAM. Konfigurasi twist_mux untuk 2 kontroller dari keyboard dan nav2. Nav2 bisa jalan namun arahnya terbalik dari goal

File: src/agv_origin_description/urdf/agv_origin.xacro (robot description, xacro)
@@ -8,5 +8,6 @@
   <parent link="base_footprint"/>
   <child link="base_link"/>
-  <origin xyz="0 0 0.1005" rpy="0 0 3.14159"/>
+  <!-- <origin xyz="0 0 0.1005" rpy="0 0 3.14159"/> -->
+  <origin xyz="0 0 0.1005" rpy="0 0 0"/>
 </joint>
 <link name="base_link">

Commit message: Fix nav2

File: src/agv_origin_description/urdf/agv_origin.xacro (robot description, xacro)
@@ -8,6 +8,6 @@
   <parent link="base_footprint"/>
   <child link="base_link"/>
-  <!-- <origin xyz="0 0 0.1005" rpy="0 0 3.14159"/> -->
-  <origin xyz="0 0 0.1005" rpy="0 0 0"/>
+  <origin xyz="0 0 0.1005" rpy="0 0 3.14159"/>
+  <!-- <origin xyz="0 0 0.1005" rpy="0 0 0"/> -->
 </joint>
 <link name="base_link">
